Commit message: divided xacro into macro + impl

File: omron_imm_description/urdf/system.urdf.xacro (robot description, xacro)
@@ -1,126 +1,6 @@
 <?xml version="1.0"?>
 <robot xmlns:xacro="http://www.ros.org/wiki/xacro" name="omron_imm">
-  <xacro:arg name="fake" default="false"/>
-  <xacro:arg name="ns" default="" />
-  <xacro:arg name="prefix" default="" />
-  <xacro:arg name="trans_hw_iface" default="hardware_interface/PositionJointInterface" />
-  <xacro:arg name="use_ros2_control_gripper" default="false"/>
-<!-- Kinematics -->
-  <link name="$(arg prefix)base_link"/>
-  <!-- LD60 -->
-  <xacro:include filename="$(find omron_description)/urdf/LD60.xacro"/>
-  <xacro:LD60  prefix="$(arg prefix)">
-    <origin xyz="0 0 0" rpy="0 0 0" />
-  </xacro:LD60>
-  <!-- TM12 -->
-  <xacro:include filename="$(find tm_description)/xacro/macro.gazebo.xacro" />
-  <xacro:include filename="$(find tm_description)/xacro/macro.transmission.xacro" />
-  <xacro:include filename="$(find tm_description)/xacro/macro.materials.xacro" />
-  <xacro:include filename="$(find tm_description)/xacro/macro.tm12-nominal.urdf.xacro"/>
-  <xacro:tmr_gazebo ns="$(arg ns)" prefix="$(arg prefix)" />
-  <xacro:tmr_transmission prefix="$(arg prefix)" hw_iface="$(arg trans_hw_iface)" />
-  <xacro:tmr_materials/>
-  <xacro:tm12 ns="$(arg ns)" prefix="$(arg prefix)" />
-  <!-- Structure between LD60 and TM12 -->
-  <xacro:property name="bar_size" value="0.9 0.03 0.03"/>
-  <material name="basic_grey">
-    <color rgba="0.5 0.5 0.5 1.0"/>
-  </material>
-  <link name="$(arg prefix)right_bar">
-    <visual>
-      <geometry>
-        <box size="${bar_size}"/>
-      </geometry>
-      <material name="basic_grey"/>
-    </visual>
-  </link>
-  <link name="$(arg prefix)left_bar">
-    <visual>
-      <geometry>
-        <box size="${bar_size}"/>
-      </geometry>
-      <material name="basic_grey"/>
-    </visual>
-  </link>
-  <link name="$(arg prefix)tm_support">
-    <visual>
-      <geometry>
-        <box size="0.3 0.3 0.02"/>
-      </geometry>
-      <material name="basic_grey"/>
-    </visual>
-  </link>
-  <link name="$(arg prefix)tm_controller">
-    <visual>
-      <geometry>
-        <box size="0.44 0.41 0.21"/>
-      </geometry>
-      <material name="black"/>
-    </visual>
-    <collision>
-      <geometry>
-        <box size="0.46 0.43 0.23"/>
-      </geometry>
-      <material name="red"/>
-    </collision>
-  </link>
-  <joint name="$(arg prefix)pose_right_bar" type="fixed">
-    <parent link="$(arg prefix)base_link"/>
-    <child link="$(arg prefix)right_bar"/>
-    <origin xyz="-0.18 0.13 0.41"/>
-  </joint>
-  <joint name="$(arg prefix)pose_left_bar" type="fixed">
-    <parent link="$(arg prefix)base_link"/>
-    <child link="$(arg prefix)left_bar"/>
-    <origin xyz="-0.18 -0.13 0.41"/>
-  </joint>
-  <joint name="$(arg prefix)pose_tm_support" type="fixed">
-    <parent link="$(arg prefix)base_link"/>
-    <child link="$(arg prefix)tm_support"/>
-    <origin xyz="0.12 0.0 0.44"/>
-  </joint>
-  <joint name="$(arg prefix)pose_tm_controller" type="fixed">
-    <parent link="$(arg prefix)left_bar"/>
-    <child  link="$(arg prefix)tm_controller"/>
-    <origin xyz="-0.26 0.13 0.12"/>
-  </joint>
-  <joint name="$(arg prefix)lifter" type="fixed">
-    <parent link="$(arg prefix)base_link"/>
-    <child link="$(arg prefix)base"/>
-    <origin xyz="0.12 -0.0 0.45" rpy=" 0 0 0"/>
-    <axis xyz="0 0 1"/>
-  </joint>
-  <!-- Force sensor and Gripper -->
-  <xacro:include filename="$(find robotiq_ft_sensor_description)/urdf/robotiq_ft300.urdf.xacro"/>
-  <xacro:include filename="$(find robotiq_description)/urdf/robotiq_2f_140_macro.urdf.xacro"/>
-  <xacro:robotiq_ft300 parent="$(arg prefix)flange" prefix="$(arg prefix)">
-    <origin xyz="0 0 0" rpy="0 0 0"/>
-  </xacro:robotiq_ft300>
-  <xacro:robotiq_gripper name="gripper" prefix="$(arg prefix)" parent="$(arg prefix)robotiq_ft_frame_id" include_ros2_control="false">
-    <origin xyz="0.0 0.0 -0.0065" rpy="0.0 0.0 0.0"/>
-  </xacro:robotiq_gripper>
-  <!-- <joint name="$(arg prefix)from_sensor_to_gripper" type="fixed"> -->
-    <!-- <origin xyz="0.0 0.0 -0.0065" rpy="0.0 0.0 ${pi/2}"/> -->
-    <!-- <parent link="$(arg prefix)robotiq_ft_frame_id"/> -->
-    <!-- <child link="$(arg prefix)robotiq_arg2f_base_link"/> -->
-  <!-- </joint> -->
-  <link name="$(arg prefix)tip"/>
-  <joint name="$(arg prefix)to_tip" type="fixed">
-    <parent link="$(arg prefix)robotiq_140_base_link"/>
-    <child link="$(arg prefix)tip"/>
-    <origin xyz="0 0 0.1767" rpy="0 0 0"/>
-  </joint>
-<!-- ros2_control -->
-  <!-- LD60 -->
-  <xacro:include filename="$(find omron_hardware_interface)/urdf/omron.ros2_control.xacro"/>
-  <xacro:omron_aria name="omron_aria" use_fake_hardware="$(arg fake)"/>
-  <!-- TM12 -->
-  <xacro:if value="$(arg fake)">
-    <xacro:include filename="$(find omron_imm_moveit_config)/config/omron_imm.ros2_control.xacro"/>
-    <xacro:omron_imm_ros2_control name="tm12" initial_positions_file="$(find omron_imm_moveit_config)/config/initial_positions.yaml"/>
-  </xacro:if>
-  <xacro:unless value="$(arg fake)">
-    <xacro:include filename="$(find tm_description)/xacro/tm12.ros2_control.xacro" />
-    <xacro:tm12_ros2_control name="tm12" prefix="$(arg prefix)" />
-  </xacro:unless>
+  <xacro:arg name="fake" default="true"/>
+  <xacro:include filename="$(find omron_imm_description)/urdf/macro_omron_imm.xacro"/>
+  <xacro:omron_imm name="omron_imm" prefix="omron/" fake="$(arg fake)"/>
 </robot>

Commit message: update urdf

File: omron_imm_description/urdf/system.urdf.xacro (robot description, xacro)
@@ -13,4 +13,5 @@
   <xacro:include filename="$(find robotiq_description)/urdf/robotiq_2f_140_macro.urdf.xacro"/>
   <!-- Force Torque Sensor -->
+  <!--
   <xacro:robotiq_ft300s parent="flange" tf_prefix="$(arg prefix)">
     <origin xyz="0 0 -0.006" rpy="0 0 0"/>
@@ -18,14 +19,16 @@
   <xacro:if value="$(arg use_ft_sensor)">
     <xacro:include filename="$(find robotiq_ft_sensor_description)/urdf/robotiq_fts.ros2_control.xacro"/>
-    <xacro:robotiq_fts_ros2_control name="$(arg prefix)omron_imm/" tf_prefix="$(arg prefix)" max_retries="1" read_rate="10"/>
+    <xacro:robotiq_fts_ros2_control name="$(arg prefix)omron/" tf_prefix="$(arg prefix)" max_retries="1" read_rate="10"/>
   </xacro:if>
+  -->
   <!-- Robotiq Gripper -->
   <!-- TODO: include gazebo -->
-  <xacro:robotiq_gripper name="azrael_gripper" prefix="$(arg prefix)" parent="$(arg prefix)robotiq_ft_frame_id" include_ros2_control="false">
-    <origin xyz="0 0 -0.00695" rpy="0 0 ${pi/2}"/>
+  <xacro:robotiq_gripper name="azrael_gripper" prefix="$(arg prefix)" parent="$(arg prefix)flange" include_ros2_control="false">
+    <!-- <origin xyz="0 0 -0.00695" rpy="0 0 ${pi/2}"/> -->
+    <origin xyz="0 0 -0.006" rpy="0 0 0"/>
   </xacro:robotiq_gripper>
   <xacro:if value="$(arg use_gripper)">
     <xacro:include filename="$(find robotiq_description)/urdf/2f_140.ros2_control.xacro"/>
-    <xacro:robotiq_gripper_ros2_control name="$(arg prefix)omron_imm/robotiq_2f_140" prefix="$(arg prefix)"/>
+    <xacro:robotiq_gripper_ros2_control name="$(arg prefix)omron/robotiq_2f_140" prefix="$(arg prefix)"/>
   </xacro:if>
   <link name="$(arg prefix)tip"/>

Commit message: update urdf

File: omron_imm_description/urdf/system.urdf.xacro (robot description, xacro)
@@ -2,11 +2,12 @@
 <robot xmlns:xacro="http://www.ros.org/wiki/xacro" name="omron_imm">
   <xacro:arg name="fake" default="true"/>
-  <xacro:arg name="prefix" default="omron/"/>
+  <xacro:arg name="prefix" default="omron"/>
   <xacro:arg name="use_ft_sensor" default="true"/>
   <xacro:arg name="use_gripper" default="true"/>
+  <xacro:property name="prefix" value="$(arg prefix)/"/>
   <xacro:include filename="$(find omron_imm_description)/urdf/omron_imm.macro.xacro"/>
   <xacro:include filename="$(find omron_imm_description)/urdf/omron_imm.ros2_control.xacro"/>
-  <xacro:omron_imm name="$(arg prefix)" fake="$(arg fake)"/>
-  <xacro:omron_imm_ros2_control prefix="$(arg prefix)" fake="$(arg fake)"/>
+  <xacro:omron_imm name="${prefix}" fake="$(arg fake)"/>
+  <xacro:omron_imm_ros2_control prefix="${prefix}" fake="$(arg fake)"/>
 <!-- Force sensor and Gripper -->
   <xacro:include filename="$(find robotiq_ft_sensor_description)/urdf/robotiq_ft300s.urdf.xacro"/>
@@ -14,15 +15,15 @@
   <!-- Force Torque Sensor -->
   <!--
-  <xacro:robotiq_ft300s parent="flange" tf_prefix="$(arg prefix)">
+  <xacro:robotiq_ft300s parent="flange" tf_prefix="${prefix}">
     <origin xyz="0 0 -0.006" rpy="0 0 0"/>
   </xacro:robotiq_ft300s>
   <xacro:if value="$(arg use_ft_sensor)">
     <xacro:include filename="$(find robotiq_ft_sensor_description)/urdf/robotiq_fts.ros2_control.xacro"/>
-    <xacro:robotiq_fts_ros2_control name="$(arg prefix)omron/" tf_prefix="$(arg prefix)" max_retries="1" read_rate="10"/>
+    <xacro:robotiq_fts_ros2_control name="${prefix}omron/" tf_prefix="${prefix}" max_retries="1" read_rate="10"/>
   </xacro:if>
   -->
   <!-- Robotiq Gripper -->
   <!-- TODO: include gazebo -->
-  <xacro:robotiq_gripper name="azrael_gripper" prefix="$(arg prefix)" parent="$(arg prefix)flange" include_ros2_control="false">
+  <xacro:robotiq_gripper name="azrael_gripper" prefix="${prefix}" parent="${prefix}flange" include_ros2_control="false">
     <!-- <origin xyz="0 0 -0.00695" rpy="0 0 ${pi/2}"/> -->
     <origin xyz="0 0 -0.006" rpy="0 0 0"/>
@@ -30,10 +31,10 @@
   <xacro:if value="$(arg use_gripper)">
     <xacro:include filename="$(find robotiq_description)/urdf/2f_140.ros2_control.xacro"/>
-    <xacro:robotiq_gripper_ros2_control name="$(arg prefix)omron/robotiq_2f_140" prefix="$(arg prefix)"/>
+    <xacro:robotiq_gripper_ros2_control name="${prefix}omron/robotiq_2f_140" prefix="${prefix}"/>
   </xacro:if>
-  <link name="$(arg prefix)tip"/>
-  <joint name="$(arg prefix)to_tip" type="fixed">
-    <parent link="$(arg prefix)robotiq_140_base_link"/>
-    <child link="$(arg prefix)tip"/>
+  <link name="${prefix}tip"/>
+  <joint name="${prefix}to_tip" type="fixed">
+    <parent link="${prefix}robotiq_140_base_link"/>
+    <child link="${prefix}tip"/>
     <origin xyz="0 0 0.1767" rpy="0 0 0"/>
   </joint>
