Commit message: replaced ft package; division xacro macro and ros2_control

File: omron_imm_description/urdf/omron_imm.macro.xacro (robot description, xacro)
@@ -2,5 +2,4 @@
 <robot xmlns:xacro="http://www.ros.org/wiki/xacro" name="omron_imm">
   <xacro:macro name="omron_imm" params="name prefix fake
-                                        gripper_ros2_control:=false
                                         use_map:=true">
   <!-- <xacro:arg name="fake" default="false"/>
@@ -92,11 +91,11 @@
   </joint>
   <!-- Force sensor and Gripper -->
-  <xacro:include filename="$(find robotiq_ft_sensor_description)/urdf/robotiq_ft300.urdf.xacro"/>
+  <xacro:include filename="$(find robotiq_ft_sensor_description)/urdf/robotiq_ft300s.urdf.xacro"/>
   <xacro:include filename="$(find robotiq_description)/urdf/robotiq_2f_140_macro.urdf.xacro"/>
-  <xacro:robotiq_ft300 parent="${prefix}flange" prefix="${prefix}">
-    <origin xyz="0 0 0" rpy="0 0 0"/>
-  </xacro:robotiq_ft300>
-  <xacro:robotiq_gripper name="robotiq_2f_140" prefix="${prefix}" parent="${prefix}robotiq_ft_frame_id" include_ros2_control="${gripper_ros2_control}" use_fake_hardware="${fake}">
-    <origin xyz="0.0 0.0 -0.0065" rpy="0.0 0.0 0.0"/>
+  <xacro:robotiq_ft300s parent="flange" tf_prefix="$(arg prefix)">
+    <origin xyz="0 0 -0.006" rpy="0 0 0"/>
+  </xacro:robotiq_ft300s>
+  <xacro:robotiq_gripper name="azrael_gripper" prefix="$(arg prefix)" parent="$(arg prefix)robotiq_ft_frame_id" include_ros2_control="false">
+    <origin xyz="0 0 -0.00695" rpy="0 0 ${pi/2}"/>
   </xacro:robotiq_gripper>
   <link name="${prefix}tip"/>
@@ -106,22 +105,4 @@
     <origin xyz="0 0 0.1767" rpy="0 0 0"/>
   </joint>
-  <!-- <joint name="${prefix}from_sensor_to_gripper" type="fixed"> -->
-    <!-- <origin xyz="0.0 0.0 -0.0065" rpy="0.0 0.0 ${pi/2}"/> -->
-    <!-- <parent link="${prefix}robotiq_ft_frame_id"/> -->
-    <!-- <child link="${prefix}robotiq_arg2f_base_link"/> -->
-  <!-- </joint> -->
-<!-- ros2_control -->
-  <!-- LD60 -->
-  <xacro:include filename="$(find omron_hardware_interface)/urdf/omron.ros2_control.xacro"/>
-  <xacro:omron_aria name="omron_aria" use_fake_hardware="${fake}"/>
-  <!-- TM12 -->
-  <xacro:if value="${fake}">
-    <xacro:include filename="$(find omron_imm_moveit_config)/config/omron_imm.ros2_control.xacro"/>
-    <xacro:omron_imm_ros2_control name="tm12" initial_positions_file="$(find omron_imm_moveit_config)/config/initial_positions.yaml"/>
-  </xacro:if>
-  <xacro:unless value="${fake}">
-    <xacro:include filename="$(find tm_description)/xacro/tm12.ros2_control.xacro" />
-    <xacro:tm12_ros2_control name="tm12" prefix="${prefix}" />
-  </xacro:unless>
 </xacro:macro>
 </robot>

File: omron_imm_description/urdf/system.urdf.xacro (robot description, xacro)
@@ -2,5 +2,10 @@
 <robot xmlns:xacro="http://www.ros.org/wiki/xacro" name="omron_imm">
   <xacro:arg name="fake" default="true"/>
-  <xacro:include filename="$(find omron_imm_description)/urdf/macro_omron_imm.xacro"/>
-  <xacro:omron_imm name="omron_imm" prefix="omron/" fake="$(arg fake)"/>
+  <xacro:arg name="prefix" default="omron/"/>
+  <xacro:arg name="use_ft_sensor" default="true"/>
+  <xacro:arg name="use_gripper" default="true"/>
+  <xacro:include filename="$(find omron_imm_description)/urdf/omron_imm.macro.xacro"/>
+  <xacro:include filename="$(find omron_imm_description)/urdf/omron_imm.ros2_control.xacro"/>
+  <xacro:omron_imm name="omron_imm" prefix="$(arg prefix)" fake="$(arg fake)"/>
+  <xacro:omron_imm_ros2_control prefix="$(arg prefix)" fake="$(arg fake)" ft_sensor="$(arg use_ft_sensor)" gripper="$(arg use_gripper)"/>
 </robot>

Commit message: update urdf

File: omron_imm_description/urdf/omron_imm.macro.xacro (robot description, xacro)
@@ -1,6 +1,5 @@
 <?xml version="1.0"?>
 <robot xmlns:xacro="http://www.ros.org/wiki/xacro" name="omron_imm">
-  <xacro:macro name="omron_imm" params="name prefix fake
-                                        use_map:=true">
+  <xacro:macro name="omron_imm" params="name fake">
   <!-- <xacro:arg name="fake" default="false"/>
   <xacro:arg name="ns" default="" />
@@ -11,5 +10,5 @@
   <!-- LD60 -->
   <xacro:include filename="$(find omron_description)/urdf/LD60.xacro"/>
-  <xacro:LD60  prefix="${prefix}" use_map="true"/>
+  <xacro:LD60  name="${name}"/>
   <!-- TM12 -->
   <xacro:include filename="$(find tm_description)/xacro/macro.gazebo.xacro" />
@@ -17,8 +16,8 @@
   <xacro:include filename="$(find tm_description)/xacro/macro.materials.xacro" />
   <xacro:include filename="$(find tm_description)/xacro/macro.tm12-nominal.urdf.xacro"/>
-  <xacro:tmr_gazebo ns="${prefix}" prefix="${prefix}" />
-  <xacro:tmr_transmission prefix="${prefix}" hw_iface="${trans_hw_iface}" />
+  <xacro:tmr_gazebo ns="${name}" prefix="${name}" />
+  <xacro:tmr_transmission prefix="${name}" hw_iface="${trans_hw_iface}" />
   <xacro:tmr_materials/>
-  <xacro:tm12 ns="${prefix}" prefix="${prefix}" />
+  <xacro:tm12 ns="${name}" prefix="${name}" />
   <!-- Structure between LD60 and TM12 -->
   <xacro:property name="bar_size" value="0.9 0.03 0.03"/>
@@ -26,5 +25,5 @@
     <color rgba="0.5 0.5 0.5 1.0"/>
   </material>
-  <link name="${prefix}right_bar">
+  <link name="${name}right_bar">
     <visual>
       <geometry>
@@ -34,5 +33,5 @@
     </visual>
   </link>
-  <link name="${prefix}left_bar">
+  <link name="${name}left_bar">
     <visual>
       <geometry>
@@ -42,5 +41,5 @@
     </visual>
   </link>
-  <link name="${prefix}tm_support">
+  <link name="${name}tm_support">
     <visual>
       <geometry>
@@ -50,5 +49,5 @@
     </visual>
   </link>
-  <link name="${prefix}tm_controller">
+  <link name="${name}tm_controller">
     <visual>
       <geometry>
@@ -64,45 +63,30 @@
     </collision>
   </link>
-  <joint name="${prefix}pose_right_bar" type="fixed">
-    <parent link="${prefix}base_link"/>
-    <child link="${prefix}right_bar"/>
+  <joint name="${name}pose_right_bar" type="fixed">
+    <parent link="${name}base_footprint"/>
+    <child link="${name}right_bar"/>
     <origin xyz="-0.18 0.13 0.41"/>
   </joint>
-  <joint name="${prefix}pose_left_bar" type="fixed">
-    <parent link="${prefix}base_link"/>
-    <child link="${prefix}left_bar"/>
+  <joint name="${name}pose_left_bar" type="fixed">
+    <parent link="${name}base_footprint"/>
+    <child link="${name}left_bar"/>
     <origin xyz="-0.18 -0.13 0.41"/>
   </joint>
-  <joint name="${prefix}pose_tm_support" type="fixed">
-    <parent link="${prefix}base_link"/>
-    <child link="${prefix}tm_support"/>
+  <joint name="${name}pose_tm_support" type="fixed">
+    <parent link="${name}base_footprint"/>
+    <child link="${name}tm_support"/>
     <origin xyz="0.12 0.0 0.44"/>
   </joint>
-  <joint name="${prefix}pose_tm_controller" type="fixed">
-    <parent link="${prefix}left_bar"/>
-    <child  link="${prefix}tm_controller"/>
+  <joint name="${name}pose_tm_controller" type="fixed">
+    <parent link="${name}left_bar"/>
+    <child  link="${name}tm_controller"/>
     <origin xyz="-0.26 0.13 0.12"/>
   </joint>
-  <joint name="${prefix}lifter" type="fixed">
-    <parent link="${prefix}base_link"/>
-    <child link="${prefix}base"/>
+  <joint name="${name}lifter" type="fixed">
+    <parent link="${name}base_footprint"/>
+    <child link="${name}base"/>
     <origin xyz="0.12 -0.0 0.45" rpy=" 0 0 0"/>
     <axis xyz="0 0 1"/>
   </joint>
-  <!-- Force sensor and Gripper -->
-  <xacro:include filename="$(find robotiq_ft_sensor_description)/urdf/robotiq_ft300s.urdf.xacro"/>
-  <xacro:include filename="$(find robotiq_description)/urdf/robotiq_2f_140_macro.urdf.xacro"/>
-  <xacro:robotiq_ft300s parent="flange" tf_prefix="$(arg prefix)">
-    <origin xyz="0 0 -0.006" rpy="0 0 0"/>
-  </xacro:robotiq_ft300s>
-  <xacro:robotiq_gripper name="azrael_gripper" prefix="$(arg prefix)" parent="$(arg prefix)robotiq_ft_frame_id" include_ros2_control="false">
-    <origin xyz="0 0 -0.00695" rpy="0 0 ${pi/2}"/>
-  </xacro:robotiq_gripper>
-  <link name="${prefix}tip"/>
-  <joint name="${prefix}to_tip" type="fixed">
-    <parent link="${prefix}robotiq_140_base_link"/>
-    <child link="${prefix}tip"/>
-    <origin xyz="0 0 0.1767" rpy="0 0 0"/>
-  </joint>
 </xacro:macro>
 </robot>

File: omron_imm_description/urdf/omron_imm.ros2_control.xacro (robot description, xacro)
@@ -1,8 +1,5 @@
 <?xml version="1.0"?>
 <robot xmlns:xacro="http://www.ros.org/wiki/xacro" name="omron_imm_ros2_control">
-  <xacro:macro name="omron_imm_ros2_control" params="prefix
-                                                     fake
-                                                     ft_sensor
-                                                     gripper">
+  <xacro:macro name="omron_imm_ros2_control" params="prefix fake">
     <!-- LD60 -->
     <xacro:include filename="$(find omron_hardware_interface)/urdf/omron.ros2_control.xacro"/>
@@ -17,15 +14,4 @@
       <xacro:tm12_ros2_control name="tm12" prefix="${prefix}" />
     </xacro:unless>
-    <!-- Force Torque Sensor -->
-    <xacro:if value="${ft_sensor}">
-      <xacro:include filename="$(find robotiq_ft_sensor_description)/urdf/robotiq_fts.ros2_control.xacro"/>
-      <xacro:robotiq_fts_ros2_control name="${prefix}omron_imm/" tf_prefix="${prefix}" max_retries="1" read_rate="10"/>
-    </xacro:if>
-    <!-- Robotiq Gripper -->
-    <!-- TODO: include gazebo -->
-    <xacro:if value="${gripper}">
-      <xacro:include filename="$(find robotiq_description)/urdf/2f_140.ros2_control.xacro"/>
-      <xacro:robotiq_gripper_ros2_control name="${prefix}omron_imm/robotiq_2f_140" prefix="${prefix}"/>
-    </xacro:if>
 </xacro:macro>
 </robot>

File: omron_imm_description/urdf/system.urdf.xacro (robot description, xacro)
@@ -7,5 +7,31 @@
   <xacro:include filename="$(find omron_imm_description)/urdf/omron_imm.macro.xacro"/>
   <xacro:include filename="$(find omron_imm_description)/urdf/omron_imm.ros2_control.xacro"/>
-  <xacro:omron_imm name="omron_imm" prefix="$(arg prefix)" fake="$(arg fake)"/>
-  <xacro:omron_imm_ros2_control prefix="$(arg prefix)" fake="$(arg fake)" ft_sensor="$(arg use_ft_sensor)" gripper="$(arg use_gripper)"/>
+  <xacro:omron_imm name="$(arg prefix)" fake="$(arg fake)"/>
+  <xacro:omron_imm_ros2_control prefix="$(arg prefix)" fake="$(arg fake)"/>
+<!-- Force sensor and Gripper -->
+  <xacro:include filename="$(find robotiq_ft_sensor_description)/urdf/robotiq_ft300s.urdf.xacro"/>
+  <xacro:include filename="$(find robotiq_description)/urdf/robotiq_2f_140_macro.urdf.xacro"/>
+  <!-- Force Torque Sensor -->
+  <xacro:robotiq_ft300s parent="flange" tf_prefix="$(arg prefix)">
+    <origin xyz="0 0 -0.006" rpy="0 0 0"/>
+  </xacro:robotiq_ft300s>
+  <xacro:if value="$(arg use_ft_sensor)">
+    <xacro:include filename="$(find robotiq_ft_sensor_description)/urdf/robotiq_fts.ros2_control.xacro"/>
+    <xacro:robotiq_fts_ros2_control name="$(arg prefix)omron_imm/" tf_prefix="$(arg prefix)" max_retries="1" read_rate="10"/>
+  </xacro:if>
+  <!-- Robotiq Gripper -->
+  <!-- TODO: include gazebo -->
+  <xacro:robotiq_gripper name="azrael_gripper" prefix="$(arg prefix)" parent="$(arg prefix)robotiq_ft_frame_id" include_ros2_control="false">
+    <origin xyz="0 0 -0.00695" rpy="0 0 ${pi/2}"/>
+  </xacro:robotiq_gripper>
+  <xacro:if value="$(arg use_gripper)">
+    <xacro:include filename="$(find robotiq_description)/urdf/2f_140.ros2_control.xacro"/>
+    <xacro:robotiq_gripper_ros2_control name="$(arg prefix)omron_imm/robotiq_2f_140" prefix="$(arg prefix)"/>
+  </xacro:if>
+  <link name="$(arg prefix)tip"/>
+  <joint name="$(arg prefix)to_tip" type="fixed">
+    <parent link="$(arg prefix)robotiq_140_base_link"/>
+    <child link="$(arg prefix)tip"/>
+    <origin xyz="0 0 0.1767" rpy="0 0 0"/>
+  </joint>
 </robot>

Commit message: fake

File: omron_imm_description/urdf/omron_imm.macro.xacro (robot description, xacro)
@@ -1,6 +1,5 @@
 <?xml version="1.0"?>
 <robot xmlns:xacro="http://www.ros.org/wiki/xacro" name="omron_imm">
-  <xacro:macro name="omron_imm" params="name fake">
-  <!-- <xacro:arg name="fake" default="false"/>
+  <xacro:macro name="omron_imm" params="name">
   <xacro:arg name="ns" default="" />
   <xacro:arg name="prefix" default="" /> -->

File: omron_imm_description/urdf/omron_imm.ros2_control.xacro (robot description, xacro)
@@ -1,14 +1,14 @@
 <?xml version="1.0"?>
 <robot xmlns:xacro="http://www.ros.org/wiki/xacro" name="omron_imm_ros2_control">
-  <xacro:macro name="omron_imm_ros2_control" params="prefix fake">
+  <xacro:macro name="omron_imm_ros2_control" params="prefix use_fake_tm use_fake_omron">
     <!-- LD60 -->
     <xacro:include filename="$(find omron_hardware_interface)/urdf/omron.ros2_control.xacro"/>
-    <xacro:omron_aria name="omron_aria" use_fake_hardware="${fake}"/>
+    <xacro:omron_aria name="omron_aria" use_fake_hardware="${use_fake_omron}"/>
     <!-- TM12 -->
-    <xacro:if value="${fake}">
+    <xacro:if value="${use_fake_tm}">
       <xacro:include filename="$(find omron_imm_moveit_config)/config/omron_imm.ros2_control.xacro"/>
       <xacro:omron_imm_ros2_control name="tm12" initial_positions_file="$(find omron_imm_moveit_config)/config/initial_positions.yaml"/>
     </xacro:if>
-    <xacro:unless value="${fake}">
+    <xacro:unless value="${use_fake_tm}">
       <xacro:include filename="$(find tm_description)/xacro/tm12.ros2_control.xacro" />
       <xacro:tm12_ros2_control name="tm12" prefix="${prefix}" />

File: omron_imm_description/urdf/system.urdf.xacro (robot description, xacro)
@@ -1,13 +1,14 @@
 <?xml version="1.0"?>
 <robot xmlns:xacro="http://www.ros.org/wiki/xacro" name="omron_imm">
-  <xacro:arg name="fake" default="true"/>
+  <xacro:arg name="use_fake_tm" default="true"/>
+  <xacro:arg name="use_fake_omron" default="true"/>
   <xacro:arg name="prefix" default="omron"/>
-  <xacro:arg name="use_ft_sensor" default="true"/>
-  <xacro:arg name="use_gripper" default="true"/>
+  <xacro:arg name="use_ft_sensor" default="false"/>
+  <xacro:arg name="use_gripper" default="false"/>
   <xacro:property name="prefix" value="$(arg prefix)/"/>
   <xacro:include filename="$(find omron_imm_description)/urdf/omron_imm.macro.xacro"/>
   <xacro:include filename="$(find omron_imm_description)/urdf/omron_imm.ros2_control.xacro"/>
-  <xacro:omron_imm name="${prefix}" fake="$(arg fake)"/>
-  <xacro:omron_imm_ros2_control prefix="${prefix}" fake="$(arg fake)"/>
+  <xacro:omron_imm name="${prefix}" />
+  <xacro:omron_imm_ros2_control prefix="${prefix}" use_fake_tm="$(arg use_fake_tm)" use_fake_omron="$(arg use_fake_omron)"/>
 <!-- Force sensor and Gripper -->
   <xacro:include filename="$(find robotiq_ft_sensor_description)/urdf/robotiq_ft300s.urdf.xacro"/>
